File: open_thermostat.kicad_pcb (KiCad board)
At the start: 2 copper layers, 100 x 100 mm, 18 parts, among them J1 HEATER, J2 SSD1306 display, J3 WS8212b led strip, J4 AC IN, K1 SANYOU_SRD_Form_C, Q1 2N2219, SW1 SW_Push, U1 WeMos_D1_mini, U2 DS18B20

Commit message: pcb fixes
Parts:
- added R3: 4.7K, Resistor_SMD:R_1206_3216Metric_Pad1.30x1.75mm_HandSolder, F.Cu at (80.2, 82.3)
- Q1: footprint Package_TO_SOT_THT:TO-92_Inline -> Package_TO_SOT_SMD:SOT-23_Handsoldering
- R1, R2, R4: footprint Resistor_THT:R_Axial_DIN0207_L6.3mm_D2.5mm_P10.16mm_Horizontal -> Resistor_SMD:R_1206_3216Metric_Pad1.30x1.75mm_HandSolder
- moved R4 5.77 mm to (80.2, 87.4)
- moved R2 5.57 mm to (80.2, 77.2), turned to 180 degrees
- moved R1 5.32 mm to (80.2, 72.1), turned to 180 degrees
- moved D2 3.40 mm to (101.3, 75.8)
- moved Q1 1.79 mm to (80.2, 66.4)
Connections:
- J3 pad 1: LED -> GND
- J3 pad 2: 5V -> LED
- J3 pad 3: GND -> 5V
Routing:
- net OUT: track 7.38 -> 23.8 mm
- net Net-(Q1-B): track 21.5 -> 11.2 mm
- net 5V: track 175.6 -> 181.5 mm
- net Net-(D2-A): track 47.9 -> 51.8 mm
- net Net-(D1-A): track 47.1 -> 48.6 mm
- net LED: track 44.5 -> 43.5 mm
- net GND: track 40.6 -> 40.9 mm, vias 4 -> 7
Other:
- board text added: "Open Thermostat rev 2 - 2025-12 https://github.com/Pimentoso/open_thermostat"
- board text removed: "Open Thermostat rev 1 - 2025-12 https://github.com/Pimentoso/open_thermostat"

Commit message: wip new version
Parts:
- removed C1: 4.7uf, Capacitor_SMD:C_1206_3216Metric_Pad1.33x1.80mm_HandSolder
- added C3: 4.7uf, Capacitor_SMD:C_1206_3216Metric_Pad1.33x1.80mm_HandSolder, F.Cu at (100.4, 75.0)
- added C4: 100nf, Capacitor_SMD:C_1206_3216Metric_Pad1.33x1.80mm_HandSolder, F.Cu at (97.5, 75.0)
- added R5: 10, Resistor_SMD:R_1206_3216Metric_Pad1.30x1.75mm_HandSolder, F.Cu at (94.6, 75.0)
- moved R3 48.1 mm to (74.4, 130.0), turned to 0 degrees
- moved R4 26.1 mm to (103.2, 75.0), turned to 90 degrees
- moved D2 6.00 mm to (101.3, 81.8)
- moved R2 5.06 mm to (81.8, 72.4), turned to -90 degrees
- moved D1 1.97 mm to (109.6, 84.0)
- moved R1 1.63 mm to (78.6, 72.4), turned to 90 degrees
- turned Q1 to 90 degrees
Connections:
- D1 pad 1: 5V -> Net-(D1-K)
- K1 pad 5: 5V -> Net-(D1-K)
- R3 pad 1: 5V -> TEMP
- R3 pad 2: GND -> 5V
- R4 pad 2: 5V -> Net-(D1-K)
- U1 pad 3: unconnected-(U1-D0-Pad3) -> BTN
- U1 pad 6: BTN -> TEMP
- U1 pad 7: TEMP -> unconnected-(U1-CS/D8-Pad7)
Routing:
- net Net-(D2-A): track 51.8 -> 7.10 mm
- net 5V: track 181.5 -> 148.2 mm
- net Net-(D1-K): track 0.00 -> 28.1 mm
- net OUT: track 23.8 -> 10.1 mm
- net Net-(Q1-B): track 11.2 -> 6.42 mm
- net TEMP: track 90.2 -> 92.7 mm
- net Net-(D1-A): track 48.6 -> 50.4 mm, vias 0 -> 1
