File: open_thermostat.kicad_sch (KiCad schematic)
At the start: 18 parts, among them J1 HEATER, J2 SSD1306 display, J3 WS8212b led strip, J4 AC IN, K1 SANYOU_SRD_Form_C, Q1 2N2219, SW1 SW_Push, U1 WeMos_D1_mini, U2 DS18B20

Commit message: pcb fixes
Parts:
- added R3: 4.7K, Resistor_SMD:R_1206_3216Metric_Pad1.30x1.75mm_HandSolder, symbol Device:R
- Q1: footprint Package_TO_SOT_THT:TO-92_Inline -> Package_TO_SOT_SMD:SOT-23_Handsoldering
- R1, R2, R4: footprint Resistor_THT:R_Axial_DIN0207_L6.3mm_D2.5mm_P10.16mm_Horizontal -> Resistor_SMD:R_1206_3216Metric_Pad1.30x1.75mm_HandSolder
Connections:
- net 5V: now also J3.3 (Pin_3), R3.1; no longer J3.2 (Pin_2)
- net GND: now also J3.1 (Pin_1), R3.2; no longer J3.3 (Pin_3)
- net LED: now also J3.2 (Pin_2); no longer J3.1 (Pin_1)
Changed lines of the file:
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@@
   (junction (at 162.56 50.8) (diameter 0) (color 0 0 0 0)
   )
+  (junction (at 45.72 100.33) (diameter 0) (color 0 0 0 0)
+  )
   (junction (at 162.56 71.12) (diameter 0) (color 0 0 0 0)
   )
@@
   )
   (junction (at 143.51 71.12) (diameter 0) (color 0 0 0 0)
+  )
+  (junction (at 45.72 92.71) (diameter 0) (color 0 0 0 0)
   )
   (junction (at 162.56 92.71) (diameter 0) (color 0 0 0 0)
@@
   (no_connect (at 106.68 59.69))
   (no_connect (at 106.68 52.07))
+  (wire (pts (xy 57.15 88.9) (xy 68.58 88.9))
+    (stroke (width 0) (type default))
+  )
   (wire (pts (xy 143.51 71.12) (xy 162.56 71.12))
     (stroke (width 0) (type default))
@@
     (stroke (width 0) (type default))
   )
+  (wire (pts (xy 57.15 92.71) (xy 57.15 88.9))
+    (stroke (width 0) (type default))
+  )
   (wire (pts (xy 170.18 53.34) (xy 170.18 49.53))
     (stroke (width 0) (type default))
@@
     (stroke (width 0) (type default))
   )
+  (wire (pts (xy 45.72 92.71) (xy 57.15 92.71))
+    (stroke (width 0) (type default))
+  )
+  (wire (pts (xy 35.56 92.71) (xy 45.72 92.71))
+    (stroke (width 0) (type default))
+  )
+  (wire (pts (xy 35.56 100.33) (xy 45.72 100.33))
+    (stroke (width 0) (type default))
+  )
   (wire (pts (xy 93.98 41.91) (xy 76.2 41.91))
     (stroke (width 0) (type default))
@@
     (stroke (width 0) (type default))
   )
+  (wire (pts (xy 45.72 100.33) (xy 57.15 100.33))
+    (stroke (width 0) (type default))
+  )
   (wire (pts (xy 140.97 50.8) (xy 143.51 50.8))
     (stroke (width 0) (type default))
@@
     (stroke (width 0) (type default))
   )
+  (wire (pts (xy 57.15 100.33) (xy 57.15 104.14))
+    (stroke (width 0) (type default))
+  )
+  (wire (pts (xy 57.15 104.14) (xy 68.58 104.14))
+    (stroke (width 0) (type default))
+  )
   (wire (pts (xy 143.51 64.77) (xy 143.51 71.12))
     (stroke (width 0) (type default))
@@
     (stroke (width 0) (type default))
   )
-  (global_label "5V" (shape input) (at 64.77 133.35 180) (fields_autoplaced)
-    (effects (font (size 1.27 1.27)) (justify right))
-    (property "Intersheetrefs" "${INTERSHEET_REFS}" (at 59.4867 133.35 0)
+  (global_label "5V" (shape input) (at 64.77 135.89 180) (fields_autoplaced)
+    (effects (font (size 1.27 1.27)) (justify right))
+    (property "Intersheetrefs" "${INTERSHEET_REFS}" (at 59.4867 135.89 0)
       (effects (font (size 1.27 1.27)) (justify right) hide)
     )
@@
     )
   )
-  (global_label "5V" (shape input) (at 68.58 88.9 90) (fields_autoplaced)
-    (effects (font (size 1.27 1.27)) (justify left))
-    (property "Intersheetrefs" "${INTERSHEET_REFS}" (at 68.58 83.6167 90)
-      (effects (font (size 1.27 1.27)) (justify left) hide)
-    )
-  )
-  (global_label "GND" (shape input) (at 64.77 135.89 180) (fields_autoplaced)
-    (effects (font (size 1.27 1.27)) (justify right))
-    (property "Intersheetrefs" "${INTERSHEET_REFS}" (at 57.9143 135.89 0)
+  (global_label "5V" (shape input) (at 35.56 92.71 180) (fields_autoplaced)
+    (effects (font (size 1.27 1.27)) (justify right))
+    (property "Intersheetrefs" "${INTERSHEET_REFS}" (at 30.2767 92.71 0)
+      (effects (font (size 1.27 1.27)) (justify right) hide)
+    )
+  )
+  (global_label "GND" (shape input) (at 64.77 130.81 180) (fields_autoplaced)
+    (effects (font (size 1.27 1.27)) (justify right))
+    (property "Intersheetrefs" "${INTERSHEET_REFS}" (at 57.9143 130.81 0)
       (effects (font (size 1.27 1.27)) (justify right) hide)
     )
@@
     )
   )
-  (global_label "LED" (shape input) (at 64.77 130.81 180) (fields_autoplaced)
-    (effects (font (size 1.27 1.27)) (justify right))
-    (property "Intersheetrefs" "${INTERSHEET_REFS}" (at 58.3377 130.81 0)
+  (global_label "LED" (shape input) (at 64.77 133.35 180) (fields_autoplaced)
+    (effects (font (size 1.27 1.27)) (justify right))
+    (property "Intersheetrefs" "${INTERSHEET_REFS}" (at 58.3377 133.35 0)
       (effects (font (size 1.27 1.27)) (justify right) hide)
     )
@@
     )
   )
-  (global_label "GND" (shape input) (at 68.58 104.14 270) (fields_autoplaced)
-    (effects (font (size 1.27 1.27)) (justify right))
-    (property "Intersheetrefs" "${INTERSHEET_REFS}" (at 68.58 110.9957 90)
+  (global_label "GND" (shape input) (at 35.56 100.33 180) (fields_autoplaced)
+    (effects (font (size 1.27 1.27)) (justify right))
+    (property "Intersheetrefs" "${INTERSHEET_REFS}" (at 28.7043 100.33 0)
       (effects (font (size 1.27 1.27)) (justify right) hide)
     )
@@
       (effects (font (size 1.27 1.27)))
     )
-    (property "Footprint" "Resistor_THT:R_Axial_DIN0207_L6.3mm_D2.5mm_P10.16mm_Horizontal" (at 143.51 83.058 90)
+    (property "Footprint" "Resistor_SMD:R_1206_3216Metric_Pad1.30x1.75mm_HandSolder" (at 143.51 83.058 90)
       (effects (font (size 1.27 1.27)) hide)
     )
@@
       (effects (font (size 1.27 1.27)))
     )
-    (property "Footprint" "Resistor_THT:R_Axial_DIN0207_L6.3mm_D2.5mm_P10.16mm_Horizontal" (at 137.16 52.578 90)
+    (property "Footprint" "Resistor_SMD:R_1206_3216Metric_Pad1.30x1.75mm_HandSolder" (at 137.16 52.578 90)
       (effects (font (size 1.27 1.27)) hide)
     )
@@
       (effects (font (size 1.27 1.27)) (justify left))
     )
-    (property "Footprint" "Package_TO_SOT_THT:TO-92_Inline" (at 165.1 83.185 0)
+    (property "Footprint" "Package_TO_SOT_SMD:SOT-23_Handsoldering" (at 165.1 83.185 0)
       (effects (font (size 1.27 1.27) italic) (justify left) hide)
     )
@@
       (effects (font (size 1.27 1.27)) (justify left))
     )
-    (property "Footprint" "Resistor_THT:R_Axial_DIN0207_L6.3mm_D2.5mm_P10.16mm_Horizontal" (at 150.622 87.63 90)
+    (property "Footprint" "Resistor_SMD:R_1206_3216Metric_Pad1.30x1.75mm_HandSolder" (at 150.622 87.63 90)
       (effects (font (size 1.27 1.27)) hide)
     )
@@
         )
       )
+    )
+  )
+  (symbol (lib_id "Device:R") (at 45.72 96.52 0) (unit 1)
+    (in_bom yes) (on_board yes) (dnp no) (fields_autoplaced)
+    (property "Reference" "R3" (at 48.26 95.25 0)
+      (effects (font (size 1.27 1.27)) (justify left))
+    )
+    (property "Value" "4.7K" (at 48.26 97.79 0)
+      (effects (font (size 1.27 1.27)) (justify left))
+    )
+    (property "Footprint" "Resistor_SMD:R_1206_3216Metric_Pad1.30x1.75mm_HandSolder" (at 43.942 96.52 90)
+      (effects (font (size 1.27 1.27)) hide)
+    )
+    (property "Datasheet" "~" (at 45.72 96.52 0)
+      (effects (font (size 1.27 1.27)) hide)
+    )
+    (pin "2")
+    (pin "1")
+    (instances
+      (project "open_thermostat"
+        (path "/ad6197e1-2429-4666-933d-b1a100668f9d"
+          (reference "R3") (unit 1)
+        )
+      )

Commit message: wip new version
Parts:
- removed C1: 4.7uf, Capacitor_SMD:C_1206_3216Metric_Pad1.33x1.80mm_HandSolder, symbol Device:C
- added C3: 4.7uf, Capacitor_SMD:C_1206_3216Metric_Pad1.33x1.80mm_HandSolder, symbol Device:C
- added C4: 100nf, Capacitor_SMD:C_1206_3216Metric_Pad1.33x1.80mm_HandSolder, symbol Device:C
- added R5: 10, Resistor_SMD:R_1206_3216Metric_Pad1.30x1.75mm_HandSolder, symbol Device:R
Connections:
- net 5V: now also R3.2, R5.1; no longer D1.1 (K), K1.5, R3.1, R4.2
- net BTN: now also U1.3 (D0); no longer U1.6 (MOSI/D7)
- net GND: now also C3.1, C4.1; no longer R3.2
- net TEMP: now also R3.1, U1.6 (MOSI/D7); no longer U1.7 (CS/D8)
- new net: C3.2, C4.2, D1.1 (K), K1.5, R4.2, R5.2
Other:
- moved on the sheet: R3, U2
